File: Line.kicad_pcb (KiCad board)
At the start: 2 copper layers, 51 parts, among them U0 TCRT5000, U1 TCRT5000, U10 TCRT5000, U11 TCRT5000, U12 TCRT5000, U13 TCRT5000, U14 TCRT5000, U15 TCRT5000, U16 CD74HC4067M, U2 TCRT5000, U3 TCRT5000, U4 TCRT5000, U5 TCRT5000, U6 TCRT5000, U7 TCRT5000, U8 TCRT5000, U9 TCRT5000

Commit message: pcb
Parts:
- removed R28: 150, Resistor_SMD:R_0805_2012Metric
- removed R32: 10K, Resistor_SMD:R_0805_2012Metric
- removed U15: TCRT5000, TCRT5000:OPTO_TCRT5000
- removed the U2 at (123.4, 89.6)
- added H1: MountingHole, MountingHole:MountingHole_2.1mm, F.Cu at (149.5, 91.0)
- added H2: MountingHole, MountingHole:MountingHole_2.1mm, F.Cu at (274.5, 91.0)
- added U0: QRE1113GR, OptoDevice:OnSemi_CASE100CY, F.Cu at (155.7, 89.5)
- U1, U10, U11, U12, U13, U14, U3, U4, U5, U6, U7, U8, U9: value TCRT5000 -> QRE1113GR; footprint TCRT5000:OPTO_TCRT5000 -> OptoDevice:OnSemi_CASE100CY
- U16: moved to B.Cu
- U2: renamed from U0; value TCRT5000 -> QRE1113GR; footprint TCRT5000:OPTO_TCRT5000 -> OptoDevice:OnSemi_CASE100CY
- moved R27 119.1 mm to (240.0, 84.5), turned to 90 degrees
- moved R24 118.8 mm to (239.0, 74.0), turned to -90 degrees
- moved R20 116.1 mm to (239.0, 70.0), turned to 90 degrees
- moved R26 115.3 mm to (237.0, 84.5), turned to 90 degrees
- moved R18 114.7 mm to (224.0, 70.0), turned to 90 degrees
- moved R29 112.1 mm to (243.0, 84.5), turned to -90 degrees
- moved R25 111.2 mm to (233.5, 84.0), turned to 90 degrees
- moved R23 110.7 mm to (231.5, 74.0), turned to -90 degrees
- moved U14 109.5 mm to (268.4, 89.5), turned to -45 degrees
- moved R19 108.1 mm to (231.5, 69.9), turned to 90 degrees
- moved R17 106.8 mm to (216.5, 70.0), turned to 90 degrees
- moved U13 102.9 mm to (261.9, 82.5), turned to -45 degrees
- moved R22 102.7 mm to (224.0, 74.0), turned to -90 degrees
- moved U11 98.9 mm to (242.6, 71.5)
- moved R30 97.8 mm to (228.8, 89.4)
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Connections:
- R1 pad 2: Net-(R1-Pad2) -> Net-(U0-A)
- R10 pad 2: Net-(R10-Pad2) -> Net-(U5-A)
- R13 pad 2: Net-(R13-Pad2) -> Net-(U6-A)
- R14 pad 2: Net-(R14-Pad2) -> Net-(U7-A)
- R17 pad 2: Net-(R17-Pad2) -> Net-(U8-A)
- R18 pad 2: Net-(R18-Pad2) -> Net-(U9-A)
- R19 pad 2: Net-(R19-Pad2) -> Net-(U10-A)
- R20 pad 2: Net-(R20-Pad2) -> Net-(U11-A)
- R25 pad 2: Net-(R25-Pad2) -> Net-(U12-A)
- R26 pad 2: Net-(R26-Pad2) -> Net-(U13-A)
- R27 pad 2: Net-(R27-Pad2) -> Net-(U14-A)
- R3 pad 2: Net-(R3-Pad2) -> Net-(U1-A)
- R7 pad 2: Net-(R7-Pad2) -> Net-(U3-A)
- R9 pad 2: Net-(R9-Pad2) -> Net-(U4-A)
Other:
- board outline added: 141 x 29 mm

Commit message: sap route
Parts:
- C1, R33: moved to B.Cu
- moved R27 63.5 mm to (267.0, 142.0), turned to 45 degrees
- moved R31 63.2 mm to (264.5, 144.5), turned to -135 degrees
- moved U16 62.9 mm to (212.5, 134.8), turned to 0 degrees
- moved H1 58.9 mm to (146.0, 149.8)
- moved R2 58.5 mm to (157.8, 144.0), turned to -45 degrees
- moved R4 58.5 mm to (165.0, 137.0), turned to -45 degrees
- moved H2 58.3 mm to (276.0, 149.2)
- moved C1 57.3 mm to (216.8, 143.8), turned to 180 degrees
- moved U0 56.6 mm to (153.0, 146.0)
- moved U1 56.5 mm to (160.7, 139.0)
- moved U2 56.5 mm to (168.4, 132.5)
- moved R10 56.5 mm to (194.0, 126.5)
- moved R11 56.5 mm to (186.5, 130.5)
- moved R12 56.5 mm to (194.0, 130.5)
- moved R13 56.5 mm to (201.5, 126.5)
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Connections:
- U1 pad 1: Net-(U0-A) -> Net-(U1-A)
- U1 pad 3: C0 -> C1
- U2 pad 1: Net-(U0-A) -> Net-(U2-A)
- U2 pad 3: C0 -> C2
Routing:
- net +3.3V: track 0.00 -> 30.0 mm
- net Net-(U0-A): track 0.00 -> 7.67 mm
- net Net-(U1-A): track 0.00 -> 7.09 mm
- net Net-(U2-A): track 0.00 -> 5.99 mm
- net C13: track 0.00 -> 5.85 mm
- net C7: track 0.00 -> 5.59 mm
- net C14: track 0.00 -> 5.44 mm
- net C12: track 0.00 -> 5.14 mm
- net C9: track 0.00 -> 5.09 mm
- net C8: track 0.00 -> 5.09 mm
- net C6: track 0.00 -> 5.09 mm
- net C5: track 0.00 -> 5.09 mm
- net C4: track 0.00 -> 5.09 mm
- net C3: track 0.00 -> 5.09 mm
- net C11: track 0.00 -> 5.09 mm
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Other:
- board size 141 x 29 mm -> 143 x 33 mm

Commit message: đon
Parts:
- added J1: Conn_01x06_Pin, Connector_JST:JST_ZH_B6B-ZR_1x06_P1.50mm_Vertical, F.Cu at (150.2, 109.8)
- moved R33 90.2 mm to (142.6, 84.3)
- moved C1 89.1 mm to (150.8, 83.8), turned to 0 degrees
- moved U16 79.2 mm to (146.1, 91.7), turned to 90 degrees
- moved H1 77.9 mm to (80.5, 107.6)
- moved R6 77.6 mm to (107.4, 88.7)
- moved R5 77.6 mm to (104.9, 86.2)
- moved U2 77.6 mm to (103.1, 90.6)
- moved H2 77.6 mm to (210.8, 107.3)
- moved R1 77.6 mm to (90.0, 99.6)
- moved R10 77.6 mm to (128.8, 84.6)
- moved R11 77.6 mm to (121.2, 88.6)
- moved R12 77.6 mm to (128.8, 88.6)
- moved R13 77.6 mm to (136.2, 84.6)
- moved R14 77.6 mm to (143.2, 84.6)
- moved R15 77.6 mm to (136.2, 88.6)
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Routing:
- net +3.3V: track 30.0 -> 272.5 mm, vias 0 -> 1
- net C14: track 5.44 -> 67.3 mm, vias 0 -> 1
- net C0: track 4.23 -> 57.3 mm, vias 0 -> 1
- net C13: track 5.85 -> 56.7 mm, vias 0 -> 1
- net C12: track 5.14 -> 51.7 mm, vias 0 -> 1
- net C1: track 3.78 -> 48.3 mm, vias 0 -> 1
- net C2: track 3.67 -> 46.8 mm, vias 0 -> 1
- net C3: track 5.09 -> 42.8 mm, vias 0 -> 1
- net C11: track 5.09 -> 35.5 mm, vias 0 -> 1
- net C4: track 5.09 -> 34.6 mm, vias 0 -> 1
- net C5: track 5.09 -> 30.1 mm, vias 0 -> 1
- net S2: track 0.00 -> 24.9 mm
- net S3: track 0.00 -> 24.8 mm
- net C10: track 5.09 -> 26.2 mm, vias 0 -> 1
- net C6: track 5.09 -> 23.0 mm, vias 0 -> 1
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- added copper zone on B.Cu, net GND
- added copper zone on F.Cu, net GND
Other:
- board size 143 x 33 mm -> 137.3 x 33 mm
- board text added: "Very good sensors"

Commit message: output gerber
Parts:
- added D1: LED, LED_SMD:LED_0603_1608Metric, F.Cu at (149.0, 105.2)
- added H1: MountingHole, MountingHole:MountingHole_2.1mm, F.Cu at (110.2, 89.2)
- added H2: MountingHole, MountingHole:MountingHole_2.1mm, F.Cu at (181.5, 89.2)
- added R34: 470, Resistor_SMD:R_0805_2012Metric, F.Cu at (151.2, 105.2)
- moved R5 1.20 mm to (103.9, 86.9)
- moved R6 1.20 mm to (106.4, 89.4)
Routing:
- net +3.3V: track 272.5 -> 278.8 mm
- net Net-(D1-A): track 0.00 -> 2.24 mm
- net Net-(U2-A): track 5.99 -> 4.71 mm
- net C2: track 46.8 -> 45.7 mm

Commit message: holes
Parts:
- moved H1 29.4 mm to (136.8, 102.0)
- moved H2 28.7 mm to (155.8, 102.0)
Other:
- board size 137.3 x 33 mm -> 137.3 x 33.2 mm
